File: as5040_v2.kicad_pcb (KiCad board)
At the start: 2 copper layers, 28 x 28 mm, 20 parts, among them J1 Conn_02x05_Odd_Even, J2 Conn_01x05_Male, J3 Conn_01x06_Male, J4 Conn_01x03_Male, U1 AS5045B

Commit message: Cleanup
Parts:
- removed the REF** at (115.0, 101.0)
- removed the REF** at (95.0, 81.0)
- added G***: LOGO, graphics:progresja_13.4x3.8mm, B.Cu at (103.0, 130.5)
- added REF**: OSHW-Logo_5.7x6mm_SilkScreen, Symbol:OSHW-Logo_5.7x6mm_SilkScreen, B.Cu at (100.0, 136.0)
- added REF**: MountingHole_3.2mm_M3, MountingHole:MountingHole_3.2mm_M3, F.Cu at (114.0, 146.0)
- added REF**: MountingHole_3.2mm_M3, MountingHole:MountingHole_3.2mm_M3, F.Cu at (94.0, 126.0)
- moved J3 45.0 mm to (92.0, 132.8)
- moved R3 45.0 mm to (112.5, 130.8)
- moved R7 45.0 mm to (112.5, 130.8)
- moved C1 45.0 mm to (97.4, 139.5)
- moved C2 45.0 mm to (95.8, 139.5)
- moved J1 45.0 mm to (113.5, 141.0)
- moved J2 45.0 mm to (106.5, 124.0)
- moved J4 45.0 mm to (102.7, 148.0)
- moved R1 45.0 mm to (112.5, 133.4)
- moved R2 45.0 mm to (112.5, 141.0)
- moved R4 45.0 mm to (112.5, 138.5)
- moved R5 45.0 mm to (112.5, 138.5)
- moved R6 45.0 mm to (112.5, 141.0)
- moved R8 45.0 mm to (112.5, 133.4)
- moved R9 45.0 mm to (99.0, 137.8)
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Other:
- board text added: "AS5045B breakout board"
- board text added: "Solder if supply 3V3"
- board text removed: "Zewrzeć jeśli zasilanie 3V3"

Commit message: New OSWH logo
Parts:
- moved REF** 4.50 mm to (100.0, 140.5)
Changed lines of the file:
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@@
   )
   (module Symbol:OSHW-Logo_5.7x6mm_SilkScreen (layer B.Cu)
-    (at 100 136 180)
+    (at 100 140.5 180)
     (descr "Open Source Hardware Logo")
     (tags "Logo OSHW")
@@
   (gr_line (start 118 122) (end 118 150) (layer Dwgs.User) (width 0.15))
   (gr_line (start 90 122) (end 118 122) (layer Dwgs.User) (width 0.15))
-  (gr_text "AS5045B \nbreakout board\n" (at 103 142) (layer B.SilkS)
+  (gr_text "AS5045B \nbreakout board\n" (at 103 135.5) (layer B.SilkS)
     (effects (font (size 1 1) (thickness 0.15)) (justify mirror))
   )
-  (gr_text 3V3 (at 106.5 138.25) (layer B.SilkS)
+  (gr_text 3V3 (at 106.7 142.25) (layer B.SilkS)
     (effects (font (size 1 1) (thickness 0.15)) (justify left mirror))
   )
-  (gr_text 5V (at 106.5 135.25) (layer B.SilkS)
+  (gr_text 5V (at 106.6 139.25) (layer B.SilkS)
     (effects (font (size 1 1) (thickness 0.15)) (justify left mirror))
   )
-  (gr_line (start 109.5 139.25) (end 109.5 137.25) (layer B.SilkS) (width 0.12))
-  (gr_line (start 107.5 139.25) (end 109.5 139.25) (layer B.SilkS) (width 0.12))
-  (gr_line (start 107.5 137.25) (end 107.5 139.25) (layer B.SilkS) (width 0.12))
-  (gr_line (start 109.5 137.25) (end 107.5 137.25) (layer B.SilkS) (width 0.12))
-  (gr_line (start 109.5 136.25) (end 109.5 134.25) (layer B.SilkS) (width 0.12))
-  (gr_line (start 107.5 136.25) (end 109.5 136.25) (layer B.SilkS) (width 0.12))
-  (gr_line (start 107.5 134.25) (end 107.5 136.25) (layer B.SilkS) (width 0.12))
-  (gr_line (start 109.5 134.25) (end 107.5 134.25) (layer B.SilkS) (width 0.12))
+  (gr_line (start 109 143.25) (end 109 141.25) (layer B.SilkS) (width 0.12))
+  (gr_line (start 107 143.25) (end 109 143.25) (layer B.SilkS) (width 0.12))
+  (gr_line (start 107 141.25) (end 107 143.25) (layer B.SilkS) (width 0.12))
+  (gr_line (start 109 141.25) (end 107 141.25) (layer B.SilkS) (width 0.12))
+  (gr_line (start 109 140.25) (end 109 138.25) (layer B.SilkS) (width 0.12))
+  (gr_line (start 107 140.25) (end 109 140.25) (layer B.SilkS) (width 0.12))
+  (gr_line (start 107 138.25) (end 107 140.25) (layer B.SilkS) (width 0.12))
+  (gr_line (start 109 138.25) (end 107 138.25) (layer B.SilkS) (width 0.12))
   (gr_line (start 108.1 140.15) (end 99.5 140.15) (layer F.SilkS) (width 0.12))
   (gr_line (start 99.5 140.15) (end 99 139.65) (layer F.SilkS) (width 0.12))
@@
     (effects (font (size 0.8 0.8) (thickness 0.15)) (justify right mirror))
   )
-  (gr_text PWM (at 104.02 146.854 90) (layer B.SilkS)
+  (gr_text PWM (at 104 146.9 90) (layer B.SilkS)
     (effects (font (size 0.8 0.8) (thickness 0.15)) (justify right mirror))
   )
